Commit message: Navigation and Localisation with amcl

File: install/rovo_ur_description/share/rovo_ur_description/urdf/kiros.xacro (robot description, xacro)
@@ -1 +1,152 @@
-/home/kevin/Desktop/rovo_ur_ws/src/rovo_ur_description/urdf/kiros.xacro
+<?xml version="1.0"?>
+<robot name="rovo_2w" xmlns:xacro="http://www.ros.org/wiki/xacro">
+  <!-- Paths injected from launch -->
+  <xacro:arg name="controllers_yaml" default=""/>
+  <xacro:arg name="mesh_file"  default="package://rovo_ur_description/meshes/rovo.dae"/>
+  <xacro:arg name="mesh_scale" default="1 1 1"/>
+  <xacro:arg name="mesh_xyz"   default="0 0.07 0.28"/>
+  <xacro:arg name="mesh_rpy"   default="-1.57079632679 0 1.57079632679"/>
+  <!-- Two-wheel (skid/diff) params -->
+  <xacro:property name="wheel_separation" value="0.80"/>
+  <xacro:property name="wheel_radius"     value="0.19"/>
+  <xacro:property name="wheel_width"      value="0.06"/>
+  <xacro:property name="wheel_x"          value="0.00"/>
+  <xacro:property name="wheel_z"          value="0.12"/>
+  <!-- Base collision shape and mass -->
+  <xacro:property name="col_l" value="1.4"/>
+  <xacro:property name="col_w" value="1.3"/>
+  <xacro:property name="col_h" value="2.0"/>
+  <xacro:property name="base_mass" value="60.0"/>
+  <!-- helpers -->
+  <xacro:property name="b"  value="${wheel_separation}"/>
+  <xacro:property name="r"  value="${wheel_radius}"/>
+  <xacro:property name="ww" value="${wheel_width}"/>
+  <xacro:property name="wx" value="${wheel_x}"/>
+  <xacro:property name="wz" value="${wheel_z}"/>
+  <!-- Massless root -->
+  <link name="base_footprint"/>
+  <joint name="base_footprint_to_base_link" type="fixed">
+    <parent link="base_footprint"/>
+    <child  link="base_link"/>
+  </joint>
+  <!-- Base link -->
+  <link name="base_link">
+    <visual>
+      <geometry><mesh filename="$(arg mesh_file)" scale="$(arg mesh_scale)"/></geometry>
+      <origin xyz="$(arg mesh_xyz)" rpy="$(arg mesh_rpy)"/>
+    </visual>
+    <!-- <collision name="base_collision">
+      <geometry><box size="${col_l} ${col_w} ${col_h}"/></geometry>
+      <origin xyz="0 0 ${col_h/2 + 0.05}"/>
+    </collision> -->
+    <collision name="left_track_skid">
+      <origin xyz="0 ${b/2.0 +0.1} 0.02" rpy="0 0 0"/>
+      <geometry>
+        <box size="${col_l*0.8} 0.05 0.03"/> </geometry>
+    </collision>
+    <collision name="right_track_skid">
+      <origin xyz="0 ${-b/2.0 - 0.1} 0.02" rpy="0 0 0"/>
+      <geometry>
+        <box size="${col_l*0.8} 0.05 0.03"/> </geometry>
+    </collision>
+    <inertial>
+      <mass value="${base_mass}"/>
+      <origin xyz="0 0 ${col_h/2}"/>
+      <inertia
+        ixx="${(1.0/12.0)*base_mass*(col_h*col_h + col_w*col_w)}"
+        iyy="${(1.0/12.0)*base_mass*(col_l*col_l + col_h*col_h)}"
+        izz="${(1.0/12.0)*base_mass*(col_l*col_l + col_w*col_w)}"
+        ixy="0" ixz="0" iyz="0"/>
+    </inertial>
+  </link>
+  <!-- left wheel -->
+  <link name="left_wheel_link">
+    <visual>
+      <geometry><cylinder length="${ww}" radius="${r}"/></geometry>
+      <origin xyz="0 0 0" rpy="1.57079632679 0 0"/>
+    </visual>
+    <collision>
+      <geometry><cylinder length="${ww}" radius="${r}"/></geometry>
+      <origin xyz="0 0 0" rpy="1.57079632679 0 0"/>
+    </collision>
+    <inertial>
+      <mass value="3.0"/>
+      <origin xyz="0 0 0"/>
+      <inertia ixx="0.02" iyy="0.02" izz="0.01" ixy="0" ixz="0" iyz="0"/>
+    </inertial>
+  </link>
+  <joint name="left_wheel_joint" type="continuous">
+    <parent link="base_link"/><child link="left_wheel_link"/>
+    <origin xyz="${wx} ${b/2.0} ${wz}" rpy="0 0 0"/>
+    <axis xyz="0 1 0"/>
+    <dynamics damping="0.02" friction="0.0"/>
+  </joint>
+  <!-- right wheel -->
+  <link name="right_wheel_link">
+    <visual>
+      <geometry><cylinder length="${ww}" radius="${r}"/></geometry>
+      <origin xyz="0 0 0" rpy="1.57079632679 0 0"/>
+    </visual>
+    <collision>
+      <geometry><cylinder length="${ww}" radius="${r}"/></geometry>
+      <origin xyz="0 0 0" rpy="1.57079632679 0 0"/>
+    </collision>
+    <inertial>
+      <mass value="3.0"/>
+      <origin xyz="0 0 0"/>
+      <inertia ixx="0.02" iyy="0.02" izz="0.01" ixy="0" ixz="0" iyz="0"/>
+    </inertial>
+  </link>
+  <joint name="right_wheel_joint" type="continuous">
+    <parent link="base_link"/><child link="right_wheel_link"/>
+    <origin xyz="${wx} ${-b/2.0} ${wz}" rpy="0 0 0"/>
+    <axis xyz="0 1 0"/>
+    <dynamics damping="0.02" friction="0.0"/>
+  </joint>
+  <!-- Rear SICK nanoScan3 -->
+  <link name="nano_scan_link"/>
+  <joint name="nano_scan_joint" type="fixed">
+    <parent link="base_link"/>
+    <child  link="nano_scan_link"/>
+    <!-- Example: 0.40 m behind base_link origin, same height, facing backwards -->
+    <origin xyz="0.50 -0.50 0.60" rpy="0 0 -0.785398"/>
+  </joint>
+ <ros2_control name="rovo_system" type="system">
+  <hardware>
+    <plugin>rovo_can_driver/RovoCanSystem</plugin>
+    <!-- Reuse existing xacro properties, no duplication of numbers -->
+    <param name="can_interface">can0</param>
+    <param name="wheel_radius">${wheel_radius}</param>
+    <param name="wheel_separation">${wheel_separation}</param>
+    <param name="gear_ratio">16.0</param>
+    <param name="max_motor_rpm">2000.0</param>
+    <param name="enable_tx">true</param>
+    <param name="external_password">MATTRO</param>
+  </hardware>
+  <joint name="left_wheel_joint">
+    <command_interface name="velocity"/>
+    <state_interface   name="position"/>
+    <state_interface   name="velocity"/>
+  </joint>
+  <joint name="right_wheel_joint">
+    <command_interface name="velocity"/>
+    <state_interface   name="position"/>
+    <state_interface   name="velocity"/>
+  </joint>
+ </ros2_control>
+  <!-- GZ system plugin: starts controller_manager inside gz and loads controllers.yaml -->
+  <gazebo>
+    <plugin filename="libgz_ros2_control-system.so"
+            name="gz_ros2_control::GazeboSimROS2ControlPlugin">
+      <parameters>$(arg controllers_yaml)</parameters>
+      <controller_manager_prefix_node_name>controller_manager</controller_manager_prefix_node_name>
+    </plugin>
+  </gazebo>
+  <gazebo reference="left_track_skid">
+      <mu1>2.0</mu1>    <mu2>0.05</mu2>   <fdir1>1 0 0</fdir1> </gazebo>
+    <gazebo reference="right_track_skid">
+      <mu1>1.5</mu1>
+      <mu2>0.05</mu2>
+      <fdir1>1 0 0</fdir1>
+    </gazebo>
+</robot>

File: install/rovo_ur_description/share/rovo_ur_description/urdf/rovo_ur.xacro (robot description, xacro)
@@ -1 +1,154 @@
-/home/kevin/Desktop/rovo_ur_ws/src/rovo_ur_description/urdf/rovo_ur.xacro
+<?xml version="1.0"?>
+<robot name="rovo_2w" xmlns:xacro="http://www.ros.org/wiki/xacro">
+  <!-- Paths injected from launch -->
+  <xacro:arg name="controllers_yaml" default=""/>
+  <xacro:arg name="mesh_file"  default="package://rovo_ur_description/meshes/rovo.dae"/>
+  <xacro:arg name="mesh_scale" default="1 1 1"/>
+  <xacro:arg name="mesh_xyz"   default="0 0.07 0.28"/>
+  <xacro:arg name="mesh_rpy"   default="-1.57079632679 0 1.57079632679"/>
+  <!-- Two-wheel (skid/diff) params -->
+  <xacro:property name="wheel_separation" value="0.80"/>
+  <xacro:property name="wheel_radius"     value="0.12"/>
+  <xacro:property name="wheel_width"      value="0.06"/>
+  <xacro:property name="wheel_x"          value="0.00"/>
+  <xacro:property name="wheel_z"          value="0.12"/>
+  <!-- Base collision shape and mass -->
+  <xacro:property name="col_l" value="1.4"/>
+  <xacro:property name="col_w" value="1.3"/>
+  <xacro:property name="col_h" value="2.0"/>
+  <xacro:property name="base_mass" value="60.0"/>
+  <!-- helpers -->
+  <xacro:property name="b"  value="${wheel_separation}"/>
+  <xacro:property name="r"  value="${wheel_radius}"/>
+  <xacro:property name="ww" value="${wheel_width}"/>
+  <xacro:property name="wx" value="${wheel_x}"/>
+  <xacro:property name="wz" value="${wheel_z}"/>
+  <!-- Massless root -->
+  <link name="base_footprint"/>
+  <joint name="base_footprint_to_base_link" type="fixed">
+    <parent link="base_footprint"/>
+    <child  link="base_link"/>
+  </joint>
+  <!-- Base link -->
+  <link name="base_link">
+    <visual>
+      <geometry><mesh filename="$(arg mesh_file)" scale="$(arg mesh_scale)"/></geometry>
+      <origin xyz="$(arg mesh_xyz)" rpy="$(arg mesh_rpy)"/>
+    </visual>
+    <!-- <collision name="base_collision">
+      <geometry><box size="${col_l} ${col_w} ${col_h}"/></geometry>
+      <origin xyz="0 0 ${col_h/2 + 0.05}"/>
+    </collision> -->
+    <collision name="left_track_skid">
+      <origin xyz="0 ${b/2.0 +0.1} 0.02" rpy="0 0 0"/>
+      <geometry>
+        <box size="${col_l*0.8} 0.05 0.03"/> </geometry>
+    </collision>
+    <collision name="right_track_skid">
+      <origin xyz="0 ${-b/2.0 - 0.1} 0.02" rpy="0 0 0"/>
+      <geometry>
+        <box size="${col_l*0.8} 0.05 0.03"/> </geometry>
+    </collision>
+    <inertial>
+      <mass value="${base_mass}"/>
+      <origin xyz="0 0 ${col_h/2}"/>
+      <inertia
+        ixx="${(1.0/12.0)*base_mass*(col_h*col_h + col_w*col_w)}"
+        iyy="${(1.0/12.0)*base_mass*(col_l*col_l + col_h*col_h)}"
+        izz="${(1.0/12.0)*base_mass*(col_l*col_l + col_w*col_w)}"
+        ixy="0" ixz="0" iyz="0"/>
+    </inertial>
+  </link>
+  <!-- left wheel -->
+  <link name="left_wheel_link">
+    <visual>
+      <geometry><cylinder length="${ww}" radius="${r}"/></geometry>
+      <origin xyz="0 0 0" rpy="1.57079632679 0 0"/>
+    </visual>
+    <collision>
+      <geometry><cylinder length="${ww}" radius="${r}"/></geometry>
+      <origin xyz="0 0 0" rpy="1.57079632679 0 0"/>
+    </collision>
+    <inertial>
+      <mass value="3.0"/>
+      <origin xyz="0 0 0"/>
+      <inertia ixx="0.02" iyy="0.02" izz="0.01" ixy="0" ixz="0" iyz="0"/>
+    </inertial>
+  </link>
+  <joint name="left_wheel_joint" type="continuous">
+    <parent link="base_link"/><child link="left_wheel_link"/>
+    <origin xyz="${wx} ${b/2.0} ${wz}" rpy="0 0 0"/>
+    <axis xyz="0 1 0"/>
+    <dynamics damping="0.02" friction="0.0"/>
+  </joint>
+  <!-- right wheel -->
+  <link name="right_wheel_link">
+    <visual>
+      <geometry><cylinder length="${ww}" radius="${r}"/></geometry>
+      <origin xyz="0 0 0" rpy="1.57079632679 0 0"/>
+    </visual>
+    <collision>
+      <geometry><cylinder length="${ww}" radius="${r}"/></geometry>
+      <origin xyz="0 0 0" rpy="1.57079632679 0 0"/>
+    </collision>
+    <inertial>
+      <mass value="3.0"/>
+      <origin xyz="0 0 0"/>
+      <inertia ixx="0.02" iyy="0.02" izz="0.01" ixy="0" ixz="0" iyz="0"/>
+    </inertial>
+  </link>
+  <joint name="right_wheel_joint" type="continuous">
+    <parent link="base_link"/><child link="right_wheel_link"/>
+    <origin xyz="${wx} ${-b/2.0} ${wz}" rpy="0 0 0"/>
+    <axis xyz="0 1 0"/>
+    <dynamics damping="0.02" friction="0.0"/>
+  </joint>
+    <!-- Front SICK microScan3 -->
+  <link name="micro_scan_link"/>
+  <joint name="micro_scan_joint" type="fixed">
+    <parent link="base_link"/>
+    <child  link="micro_scan_link"/>
+    <!-- xyz in meters, rpy in radians -->
+    <!-- Example: 0.40 m in front of base_link origin, 0.30 m high -->
+    <origin xyz="0.40 0.00 0.30" rpy="0 0 0"/>
+  </joint>
+  <!-- Rear SICK nanoScan3 -->
+  <link name="nano_scan_link"/>
+  <joint name="nano_scan_joint" type="fixed">
+    <parent link="base_link"/>
+    <child  link="nano_scan_link"/>
+    <!-- Example: 0.40 m behind base_link origin, same height, facing backwards -->
+    <origin xyz="-0.40 0.00 0.30" rpy="0 0 3.14159"/>
+  </joint>
+  <!-- ros2_control: gz-sim system -->
+  <ros2_control name="rovo_system" type="system">
+    <hardware>
+      <plugin>gz_ros2_control/GazeboSimSystem</plugin>
+    </hardware>
+    <joint name="left_wheel_joint">
+      <command_interface name="velocity"/>
+      <state_interface   name="position"/>
+      <state_interface   name="velocity"/>
+    </joint>
+    <joint name="right_wheel_joint">
+      <command_interface name="velocity"/>
+      <state_interface   name="position"/>
+      <state_interface   name="velocity"/>
+    </joint>
+  </ros2_control>
+  <!-- GZ system plugin: starts controller_manager inside gz and loads controllers.yaml -->
+  <gazebo>
+    <plugin filename="libgz_ros2_control-system.so"
+            name="gz_ros2_control::GazeboSimROS2ControlPlugin">
+      <parameters>$(arg controllers_yaml)</parameters>
+      <controller_manager_prefix_node_name>controller_manager</controller_manager_prefix_node_name>
+    </plugin>
+  </gazebo>
+  <gazebo reference="left_track_skid">
+      <mu1>2.0</mu1>    <mu2>0.05</mu2>   <fdir1>1 0 0</fdir1> </gazebo>
+    <gazebo reference="right_track_skid">
+      <mu1>1.5</mu1>
+      <mu2>0.05</mu2>
+      <fdir1>1 0 0</fdir1>
+    </gazebo>
+</robot>

File: src/rovo_ur_description/urdf/kiros.xacro (robot description, xacro)
@@ -9,5 +9,5 @@
   <!-- Two-wheel (skid/diff) params -->
   <xacro:property name="wheel_separation" value="0.80"/>
-  <xacro:property name="wheel_radius"     value="0.12"/>
+  <xacro:property name="wheel_radius"     value="0.19"/>
   <xacro:property name="wheel_width"      value="0.06"/>
   <xacro:property name="wheel_x"          value="0.00"/>
@@ -104,4 +104,12 @@
     <dynamics damping="0.02" friction="0.0"/>
   </joint>
+  <!-- Rear SICK nanoScan3 -->
+  <link name="nano_scan_link"/>
+  <joint name="nano_scan_joint" type="fixed">
+    <parent link="base_link"/>
+    <child  link="nano_scan_link"/>
+    <!-- Example: 0.40 m behind base_link origin, same height, facing backwards -->
+    <origin xyz="0.50 -0.50 0.60" rpy="0 0 -0.785398"/>
+  </joint>
  <ros2_control name="rovo_system" type="system">
   <hardware>

File: src/rovo_ur_description/urdf/rovo_ur.xacro (robot description, xacro)
@@ -104,4 +104,21 @@
     <dynamics damping="0.02" friction="0.0"/>
   </joint>
+    <!-- Front SICK microScan3 -->
+  <link name="micro_scan_link"/>
+  <joint name="micro_scan_joint" type="fixed">
+    <parent link="base_link"/>
+    <child  link="micro_scan_link"/>
+    <!-- xyz in meters, rpy in radians -->
+    <!-- Example: 0.40 m in front of base_link origin, 0.30 m high -->
+    <origin xyz="0.40 0.00 0.30" rpy="0 0 0"/>
+  </joint>
+  <!-- Rear SICK nanoScan3 -->
+  <link name="nano_scan_link"/>
+  <joint name="nano_scan_joint" type="fixed">
+    <parent link="base_link"/>
+    <child  link="nano_scan_link"/>
+    <!-- Example: 0.40 m behind base_link origin, same height, facing backwards -->
+    <origin xyz="-0.40 0.00 0.30" rpy="0 0 3.14159"/>
+  </joint>
   <!-- ros2_control: gz-sim system -->
   <ros2_control name="rovo_system" type="system">
